File: LogicBoard.brd (EAGLE design)
At the start: 60 x 40 mm, 87 parts, among them CON1 JST_XH_254_3THT, CON2 JST_XH_254_3THT, IC1 TL074SOIC14, IC2 LM317SOT223, IC3 TL074SOIC14, IC4 TL074SOIC14, J1 SJ-3524-SMT-TR, J2 PJRAN1X1U01X, J3 PJRAN1X1U01X

Commit message: shematic finished
Parts:
- removed CON1: JST_XH_254_3THT, LARS_CONN v48:JST_XH_254_3_THT
- added AUDIO_OUT_R: JST_XH_254_3THT, LARS_CONN v48:JST_XH_254_3_THT
- added C26, C27, C28, C31: 0u1/6V3, rcl:C1206
- added C29, C32: 1u/6V3, rcl:C1206
- added C30, C33: 10u/6V3, rcl:C1206
- added D1, D2, D3, D4, D5: DIODE_PGB-0603MP, 52101-101-REV-A_v16:DIODE_PGB-0603MP
- added R53: 5k1, rcl:R0603
- added R54: 2K4, rcl:R0603
- added R55: 0, rcl:R0603
- R12, R14, R17, R52: value (none) -> 100K
- R13, R15, R16: value (none) -> 0
- renumbered CON2 to AUDIO_OUT_L, J1 to LINE_IN, J2 to IN_R, J3 to IN_L
Connections:
- net VREF_2V5 renamed VREF_2V
- removed net AVCC_5V: C12.1, C13.1, C14.1, C19.1, C20.1, C21.1, C23.1, C24.1, C25.1, IC1.4, IC3.4, IC4.4, R10.2
- removed net IN: IC2.3
- removed net OUT: IC2.2
- removed net VCC: PWR_USB.1
- new net AVCC_4V: C12.1, C13.1, C14.1, C19.1, C20.1, C21.1, C23.1, C24.1, C25.1, C28.1, C29.1, C30.1, IC1.4, IC2.2, IC3.4, IC4.4, R10.2, R54.2
- new net LINE_IN_R: R1.1-3, R12.2, R52.2
- new net N$37: AUDIO_OUT_R.P$3, C27.2
- new net N$38: PWR_USB.2, PWR_USB.3
- new net N$41: C31.1, C32.1, C33.1, D5.2, IC2.3, PWR_USB.1
- new net N$42: R1.2-2, R55.1
- new net N$43: IC2.1, R53.2, R54.1
- new net N$44: AUDIO_OUT_L.P$3, C26.2
- net AUDIO_L_N: now also AUDIO_OUT_L.P$1, D2.2
- net AUDIO_L_P: now also AUDIO_OUT_L.P$2, D1.2
- net AUDIO_R_N: now also AUDIO_OUT_R.P$1, D4.2
- net AUDIO_R_P: now also AUDIO_OUT_R.P$2, D3.2
- net GND: now also C26.1, C27.1, C28.2, C29.2, C30.2, C31.2, C32.2, C33.2, D1.1, D2.1, D3.1, D4.1, D5.1, PWR_USB.SH1, PWR_USB.SH2, R13.2, R15.2, R16.2, R53.1
- net LINE_IN_L: now also R14.2, R17.2; no longer R1.1-3
- net N$3: now also R55.2; no longer R1.2-2
Routing:
- net AVCC_5V: track 16.9 -> 0.00 mm
- net AVCC_4V: track 0.00 -> 16.9 mm

Commit message: rev1 complete - DRC runs without errors
Parts:
- removed AUDIO_OUT_L, AUDIO_OUT_R: JST_XH_254_3THT, LARS_CONN v48:JST_XH_254_3_THT
- removed IN_L, IN_R: PJRAN1X1U01X, Connector:PJRAN1X1U01X
- removed LINE_IN: SJ-3524-SMT-TR, Audio Connectors:SJ-3524-SMT-TR
- removed PWR_USB: 61729-1011, Connector_USB:61729-1011BLF
- added CON1, CON2: JST_XH_254_3THT, LARS_CONN v48:JST_XH_254_3_THT
- added J1: SJ-3524-SMT-TR, Audio Connectors:SJ-3524-SMT-TR
- added J2, J3: PJRAN1X1U01X, Connector:PJRAN1X1U01X
- added J4: 61729-1011, Connector_USB:61729-1011BLF
- C1: value 10u -> 0u1/6V3
- C10, C23: value 0u1/6V3 -> 1u/6V3
- C11, C12, C16, C17: value 0u1/6V3 -> 3u3
- C13, C24: value 1u/6V3 -> 10u/6V3
- C14: value 10u/6V3 -> 1u6
- C15: value 0u1/6V3 -> 1u6
- C2: value 10u -> 1u/6V3
- C20, C29, C32: value 1u/6V3 -> 0u1/6V3
- C21, C25, C33: value 10u/6V3 -> 0u1/6V3
- C22, C4: value 3u3 -> 0u1/6V3
- C3, C6: value 1u6 -> 10u/6V3
- C30: value 10u/6V3 -> 1u/6V3
- C31: value 0u1/6V3 -> 10u/6V3
- C5: value 3u3 -> 1u/6V3
- C7: value 3u3 -> 10u
- C8: value 0u1/6V3 -> 10u
- IC1: value TL074SOIC14 -> LM317SOT223; device LARS_AUDIO:SOIC127P600X175-14N -> LARS_POWER:SOT230P700X180-4N
- IC2: value LM317SOT223 -> TL074SOIC14; device LARS_POWER:SOT230P700X180-4N -> LARS_AUDIO:SOIC127P600X175-14N
- R1, R2: value b2k -> 0; device pot:3RP/1610G -> rcl:R0603
- R10: value 100k -> b2k; device rcl:R0603 -> pot:3RP/1610G
- R11: value 0 -> b2k; device rcl:R0603 -> pot:3RP/1610G
- R12, R52: value 100K -> 100k
- R13: value 0 -> 100k
- R14: value 100K -> 0
- R16: value 0 -> 2k
- R17: value 100K -> 2k
- R18: value 100k -> 1k
- R19: value 150k -> 1k
- R20: value 200k -> 2k
- R21: value 100k -> 2k
- R22, R39: value 100k -> 200k
- R24, R41: value 100 -> 200k
- R26, R43: value 100k -> 150k
- R3, R4, R6: value 2k -> 100K
- R30, R47: value 100 -> 100k
- R34, R51: value 200k -> 100k
- R36: value 150k -> 100k
- R37: value 200k -> 100
- R38: value 100k -> 100
- R5: value 1k -> 100K
- R53: value 5k1 -> 100k
- R54: value 2K4 -> 100
- R55: value 0 -> 100
- R7: value 2k -> 0
- R8: value 1k -> 2K4
- R9: value 100k -> 5k1
- moved R55 318.4 mm to (53.8, 33.0)
- moved R53 309.8 mm to (50.8, 35.1)
- moved R54 307.9 mm to (53.8, 25.9)
- moved C32 299.5 mm to (56.9, 25.4), turned to 90 degrees
- moved C33 299.0 mm to (56.9, 31.5), turned to 90 degrees
- moved C31 284.4 mm to (37.1, 33.0), turned to 180 degrees
- moved C29 275.2 mm to (37.1, 29.0), turned to 180 degrees
- moved D4 274.0 mm to (69.1, 27.9), turned to 180 degrees
- moved C30 271.3 mm to (37.1, 31.0), turned to 180 degrees
- moved D5 268.1 mm to (69.1, 15.7), turned to 180 degrees
- moved C28 258.4 mm to (33.0, 24.9), turned to 180 degrees
- moved D3 255.6 mm to (69.1, 17.8), turned to 180 degrees
- moved D2 254.8 mm to (69.1, 29.5), turned to 180 degrees
- moved C27 253.6 mm to (33.0, 35.1), turned to 180 degrees
- moved D1 252.2 mm to (53.3, 44.2)
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Connections:
- net AUDIO_L: now also C17.2, C20.2, C21.2, R21.2; no longer C5.2, C8.2, C9.2, R4.2
- net AUDIO_L_N: now also C26.1, CON2.P$1, D3.2; no longer AUDIO_OUT_L.P$1, C11.1, D2.2
- net AUDIO_L_P: now also C25.1, CON2.P$2, D5.2; no longer AUDIO_OUT_L.P$2, C10.1, D1.2
- net AUDIO_R: now also C27.2, C28.2, R20.2; no longer C15.2, C22.2, R7.2
- net AUDIO_R_N: now also C33.1, CON1.P$1, D2.2; no longer AUDIO_OUT_R.P$1, C18.1, D4.2
- net AUDIO_R_P: now also C32.1, CON1.P$2, D4.2; no longer AUDIO_OUT_R.P$2, C17.1, D3.2
- net AVCC_4V: now also C10.1, C22.1, C31.1, C4.1, C5.1, C6.1, C9.1, IC1.2, IC2.4, R12.2, R8.2; no longer C12.1, C14.1, C19.1, C20.1, C21.1, C25.1, C28.1, IC1.4, IC2.2, R10.2, R54.2
- net FB_AUDIO_L_N: now also C26.2, R31.2, R32.1, R38.2; no longer C11.2, R26.1, R27.2, R30.2
- net FB_AUDIO_L_P: now also C25.2, R34.1, R37.2; no longer C10.2, R24.2, R32.1
- net FB_AUDIO_R_N: now also C33.2, R48.2, R49.1, R55.2; no longer C18.2, R43.1, R44.2, R47.2
- net FB_AUDIO_R_P: now also C32.2, R51.1, R54.2; no longer C17.2, R41.2, R49.1
- net GND: now also C1.2, C10.2, C15.2, C18.1, C19.1, C2.2, C22.2, C4.2, C5.2, C9.2, IC2.10, IC2.11, IC2.12, J4.4, J4.SH1, J4.SH2, R1.2, R13.1, R18.1, R19.1, R2.2, R7.2; no longer C12.2, C19.2, C20.2, C21.2, C25.2, C26.1, C27.1, C28.2, C32.2, C33.2, IC1.11, IC4.10, IC4.12, PWR_USB.4, PWR_USB.SH1, PWR_USB.SH2, R13.2, R15.2, R16.2, R5.1, R53.1, R8.1
- net L: now also J1.3, R6.1; no longer LINE_IN.3, R17.1
- net LINE_IN_L: now also R11.1-3, R3.2, R6.2; no longer R14.2, R17.2, R2.1-3
- net LINE_IN_R: now also R10.1-3, R4.2, R5.2; no longer R1.1-3, R12.2, R52.2
- net N$1: now also C8.1, IC2.9, R11.1-2, R11.2-1; no longer C1.1, IC4.9, R1.1-2, R1.2-1
- net N$10: now also J2.2, J2.3, R4.1; no longer IN_R.2, IN_R.3, R12.1
- net N$11: now also J3.2, J3.3, R3.1; no longer IN_L.2, IN_L.3, R14.1
- net N$12: now also IC2.2, R12.1, R13.2; no longer IC4.2, R10.1, R9.2
- net N$13: now also IC3.6, R23.2, R26.1; no longer IC1.6, R18.2, R19.1
- net N$14: now also IC3.2, R22.2, R25.1; no longer IC1.2, R20.2, R21.1
- net N$15: now also IC3.9, R27.2, R35.1; no longer IC1.9, R22.2, R23.1
- net N$16: now also IC3.8, R35.2, R37.1; no longer IC1.8, R23.2, R24.1
- net N$17: now also IC3.10, R28.2, R31.1; no longer IC1.10, R25.2, R27.1
- net N$18: now also IC3.13, R29.2, R36.1; no longer IC1.13, R28.2, R29.1
- net N$19: now also IC3.14, R36.2, R38.1; no longer IC1.14, R29.2, R30.1
- net N$2: now also C7.1, IC2.13, R10.1-2, R10.2-1; no longer C2.1, IC4.13, R2.1-2, R2.2-1
- net N$20: now also IC3.12, R30.2; no longer IC1.12, R31.2
- net N$21: now also IC3.1, R25.2, R29.1; no longer IC1.1, R21.2, R25.1
- net N$22: now also IC3.7, R26.2, R27.1, R30.1; no longer IC1.7, R19.2, R22.1, R31.1
- net N$23: now also C20.1, IC3.3, R24.2; no longer C8.1, IC1.3, R34.2
- net N$24: now also C21.1, R23.1; no longer C9.1, R18.1
- net N$25: now also IC4.6, R40.2, R43.1; no longer IC3.6, R35.2, R36.1
- net N$26: now also IC4.2, R39.2, R42.1; no longer IC3.2, R37.2, R38.1
- net N$27: now also IC4.9, R44.2, R52.1; no longer IC3.9, R39.2, R40.1
- net N$28: now also IC4.8, R52.2, R54.1; no longer IC3.8, R40.2, R41.1
- net N$29: now also IC4.10, R45.2, R48.1; no longer IC3.10, R42.2, R44.1
- net N$3: now also C12.1, C8.2, IC2.8, R14.2, R17.1; no longer C1.2, C7.1, IC4.8, R55.2, R6.1
- net N$30: now also IC4.13, R46.2, R53.1; no longer IC3.13, R45.2, R46.1
- net N$31: now also IC4.14, R53.2, R55.1; no longer IC3.14, R46.2, R47.1
- net N$32: now also IC4.12, R47.2; no longer IC3.12, R48.2
- net N$33: now also IC4.1, R42.2, R46.1; no longer IC3.1, R38.2, R42.1
- net N$34: now also IC4.7, R43.2, R44.1, R47.1; no longer IC3.7, R36.2, R39.1, R48.1
- net N$35: now also C27.1, IC4.3, R41.2; no longer C15.1, IC3.3, R51.2
- net N$36: now also C28.1, R40.1; no longer C16.1, R35.1
- net N$37: now also C18.2, CON1.P$3; no longer AUDIO_OUT_R.P$3, C27.2
- net N$38: now also J4.2, J4.3; no longer PWR_USB.2, PWR_USB.3
- net N$39: now also J3.1, R2.1; no longer IN_L.1, R15.1
- net N$4: now also C11.1, C7.2, IC2.14, R15.2, R16.1; no longer C2.2, C4.1, IC4.14, R11.2, R3.1
- net N$40: now also J2.1, R1.1; no longer IN_R.1, R13.1
- net N$41: now also C1.1, C2.1, C3.1, D1.2, IC1.3, J4.1; no longer C31.1, C32.1, C33.1, D5.2, IC2.3, PWR_USB.1
- net N$42: now also R11.2-2, R14.1; no longer R1.2-2, R55.1
- net N$43: now also IC1.1, R8.1, R9.2; no longer IC2.1, R53.2, R54.1
- net N$44: now also C19.2, CON2.P$3; no longer AUDIO_OUT_L.P$3, C26.2
- net N$5: now also C14.1, R16.2, R20.1; no longer C3.1, R3.2, R4.1
- net N$6: now also R10.2-2, R15.1; no longer R11.1, R2.2-2
- net N$7: now also C15.1, R17.2, R21.1; no longer C6.1, R6.2, R7.1
- net N$8: now also C11.2, C16.1, R18.2; no longer C4.2, C5.1, R5.2
- net N$9: now also C12.2, C17.1, R19.2; no longer C22.1, C7.2, R8.2
- net R: now also J1.2, J1.4, R5.1; no longer LINE_IN.2, LINE_IN.4, R52.1
- net SCHIRMUNG: now also J1.1, R7.1; no longer LINE_IN.1, R16.1
- net VREF_2V: now also IC2.1, IC2.3, IC4.5, R22.1, R24.1, R34.2, R39.1, R41.1, R51.2; no longer IC1.5, IC4.1, IC4.3, R20.1, R26.2, R34.1, R37.1, R43.2, R51.1
Routing:
- net AVCC_4V: track 16.9 -> 138.8 mm, vias 0 -> 7
- net LINE_IN_L: track 0.00 -> 71.7 mm
- net LINE_IN_R: track 0.00 -> 39.2 mm
- net N$2: track 0.00 -> 32.5 mm
- net VREF_2V: track 97.0 -> 118.3 mm, vias 6 -> 8
- net N$1: track 0.00 -> 21.0 mm
- net N$40: track 0.00 -> 19.7 mm
- net N$41: track 0.00 -> 19.4 mm
- net AUDIO_L: track 0.00 -> 18.3 mm
- net AUDIO_R: track 0.00 -> 18.0 mm
- net L: track 0.00 -> 17.9 mm
- net N$4: track 0.00 -> 16.5 mm
- net N$39: track 0.00 -> 15.2 mm
- net N$3: track 0.00 -> 14.9 mm
- net AUDIO_R_P: track 0.00 -> 13.5 mm
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- added copper zone on layer 1, net GND
- added copper zone on layer 16, net GND
Other:
- board size 60 x 40 mm -> 72 x 60 mm
- board text added: "designed by brokulp https://github.com/BrokuLP LineToBalancedAdapter-rev1"
