File: LogicBoard.sch (EAGLE design)
At the start: 87 parts, among them CON1 JST_XH_254_3THT, CON2 JST_XH_254_3THT, IC1 TL074SOIC14, IC2 LM317SOT223, IC3 TL074SOIC14, IC4 TL074SOIC14, J1 SJ-3524-SMT-TR, J2 PJRAN1X1U01X, J3 PJRAN1X1U01X

Commit message: shematic finished
Parts:
- removed CON1, CON2: JST_XH_254_3THT, LARS_CONN v48:JST_XH_254_3THT
- removed J1: SJ-3524-SMT-TR, Audio Connectors:SJ-3524-SMT-TR
- removed J2, J3: PJRAN1X1U01X, Connector:PJRAN1X1U01X
- added AUDIO_OUT_L, AUDIO_OUT_R: JST_XH_254_3THT, LARS_CONN v48:JST_XH_254_3THT
- added C26, C27, C28, C31: 0u1/6V3, rcl:C-EUC1206
- added C29, C32: 1u/6V3, rcl:C-EUC1206
- added C30, C33: 10u/6V3, rcl:C-EUC1206
- added D1, D2, D3, D4, D5: DIODE_PGB-0603MP, 52101-101-REV-A_v16:DIODE_PGB-0603MP
- added IN_L, IN_R: PJRAN1X1U01X, Connector:PJRAN1X1U01X
- added LINE_IN: SJ-3524-SMT-TR, Audio Connectors:SJ-3524-SMT-TR
- added R53: 5k1, rcl:R-EU_R0603
- added R54: 2K4, rcl:R-EU_R0603
- added R55: 0, rcl:R-EU_R0603
- R12, R14, R17, R52: value (none) -> 100K
- R13, R15, R16: value (none) -> 0
Connections:
- net VREF_2V5 renamed VREF_2V
- removed net AVCC_5V: C12.1, C13.1, C14.1, C19.1, C20.1, C21.1, C23.1, C24.1, C25.1, IC1G$1.VCC, IC3G$1.VCC, IC4G$1.VCC, R10.2
- new net AVCC_4V: C12.1, C13.1, C14.1, C19.1, C20.1, C21.1, C23.1, C24.1, C25.1, C28.1, C29.1, C30.1, IC1G$1.VCC, IC2.OUT, IC3G$1.VCC, IC4G$1.VCC, R10.2, R54.2
- new net LINE_IN_R: R1/1.E, R12.2, R52.2
- new net N$37: AUDIO_OUT_R.P$3, C27.2
- new net N$38: PWR_USB.D+, PWR_USB.D-
- new net N$41: C31.1, C32.1, C33.1, D5.2, IC2.IN, PWR_USB.VCC
- new net N$42: R1/2.S, R55.1
- new net N$43: IC2.FB, R53.2, R54.1
- new net N$44: AUDIO_OUT_L.P$3, C26.2
- net AUDIO_L_N: now also AUDIO_OUT_L.P$1, D2.2
- net AUDIO_L_P: now also AUDIO_OUT_L.P$2, D1.2
- net AUDIO_R_N: now also AUDIO_OUT_R.P$1, D4.2
- net AUDIO_R_P: now also AUDIO_OUT_R.P$2, D3.2
- net GND: now also C26.1, C27.1, C28.2, C29.2, C30.2, C31.2, C32.2, C33.2, D1.1, D2.1, D3.1, D4.1, D5.1, PWR_USB.GND, PWR_USB.SHIELD1, PWR_USB.SHIELD2, R13.2, R15.2, R16.2, R53.1
- net L: now also LINE_IN.3; no longer J1.3
- net LINE_IN_L: now also R14.2, R17.2; no longer R1/1.E
- net N$10: now also IN_R.2, IN_R.3; no longer J2.2, J2.3
- net N$11: now also IN_L.2, IN_L.3; no longer J3.2, J3.3
- net N$3: now also R55.2; no longer R1/2.S
- net N$39: now also IN_L.1; no longer J3.1
- net N$40: now also IN_R.1; no longer J2.1
- net R: now also LINE_IN.2, LINE_IN.4; no longer J1.2, J1.4
- net SCHIRMUNG: now also LINE_IN.1; no longer J1.1
Other:
- moved on the sheet: IC2, PWR_USB, R10, R12, R13, R14, R15, R16, R17, R52, R9

Commit message: rev1 complete - DRC runs without errors
Parts:
- C1: value 10u -> 0u1/6V3
- C10, C23: value 0u1/6V3 -> 1u/6V3
- C11, C12, C16, C17: value 0u1/6V3 -> 3u3
- C13, C24: value 1u/6V3 -> 10u/6V3
- C14: value 10u/6V3 -> 1u6
- C15: value 0u1/6V3 -> 1u6
- C2: value 10u -> 1u/6V3
- C20, C29, C32: value 1u/6V3 -> 0u1/6V3
- C21, C25, C33: value 10u/6V3 -> 0u1/6V3
- C22, C4: value 3u3 -> 0u1/6V3
- C3, C6: value 1u6 -> 10u/6V3
- C30: value 10u/6V3 -> 1u/6V3
- C31: value 0u1/6V3 -> 10u/6V3
- C5: value 3u3 -> 1u/6V3
- C7: value 3u3 -> 10u
- C8: value 0u1/6V3 -> 10u
- IC1: value TL074SOIC14 -> LM317SOT223; device LARS_AUDIO:TL074SOIC14 -> LARS_POWER:LM317SOT223
- IC2: value LM317SOT223 -> TL074SOIC14; device LARS_POWER:LM317SOT223 -> LARS_AUDIO:TL074SOIC14
- R1, R2: value b2k -> 0; device pot:3RP/1610G -> rcl:R-EU_R0603
- R10: value 100k -> b2k; device rcl:R-EU_R0603 -> pot:3RP/1610G
- R11: value 0 -> b2k; device rcl:R-EU_R0603 -> pot:3RP/1610G
- R12, R52: value 100K -> 100k
- R13: value 0 -> 100k
- R14: value 100K -> 0
- R16: value 0 -> 2k
- R17: value 100K -> 2k
- R18: value 100k -> 1k
- R19: value 150k -> 1k
- R20: value 200k -> 2k
- R21: value 100k -> 2k
- R22, R39: value 100k -> 200k
- R24, R41: value 100 -> 200k
- R26, R43: value 100k -> 150k
- R3, R4, R6: value 2k -> 100K
- R30, R47: value 100 -> 100k
- R34, R51: value 200k -> 100k
- R36: value 150k -> 100k
- R37: value 200k -> 100
- R38: value 100k -> 100
- R5: value 1k -> 100K
- R53: value 5k1 -> 100k
- R54: value 2K4 -> 100
- R55: value 0 -> 100
- R7: value 2k -> 0
- R8: value 1k -> 2K4
- R9: value 100k -> 5k1
- renumbered AUDIO_OUT_L to CON2, AUDIO_OUT_R to CON1, IN_L to J3, IN_R to J2, LINE_IN to J1, PWR_USB to J4
Connections:
- net AUDIO_L: now also C17.2, C20.2, C21.2, R21.2; no longer C5.2, C8.2, C9.2, R4.2
- net AUDIO_L_N: now also C26.1, D3.2; no longer C11.1, D2.2
- net AUDIO_L_P: now also C25.1, D5.2; no longer C10.1, D1.2
- net AUDIO_R: now also C27.2, C28.2, R20.2; no longer C15.2, C22.2, R7.2
- net AUDIO_R_N: now also C33.1, D2.2; no longer C18.1, D4.2
- net AUDIO_R_P: now also C32.1, D4.2; no longer C17.1, D3.2
- net AVCC_4V: now also C10.1, C22.1, C31.1, C4.1, C5.1, C6.1, C9.1, IC1.OUT, IC2G$1.VCC, R12.2, R8.2; no longer C12.1, C14.1, C19.1, C20.1, C21.1, C25.1, C28.1, IC1G$1.VCC, IC2.OUT, R10.2, R54.2
- net FB_AUDIO_L_N: now also C26.2, R31.2, R32.1, R38.2; no longer C11.2, R26.1, R27.2, R30.2
- net FB_AUDIO_L_P: now also C25.2, R34.1, R37.2; no longer C10.2, R24.2, R32.1
- net FB_AUDIO_R_N: now also C33.2, R48.2, R49.1, R55.2; no longer C18.2, R43.1, R44.2, R47.2
- net FB_AUDIO_R_P: now also C32.2, R51.1, R54.2; no longer C17.2, R41.2, R49.1
- net GND: now also C1.2, C10.2, C15.2, C18.1, C19.1, C2.2, C22.2, C4.2, C5.2, C9.2, IC2G$1.VSS, IC2G$3.IN+, IC2G$4.IN+, R1.2, R13.1, R18.1, R19.1, R2.2, R7.2; no longer C12.2, C19.2, C20.2, C21.2, C25.2, C26.1, C27.1, C28.2, C32.2, C33.2, IC1G$1.VSS, IC4G$3.IN+, IC4G$4.IN+, R13.2, R15.2, R16.2, R5.1, R53.1, R8.1
- net L: now also R6.1; no longer R17.1
- net LINE_IN_L: now also R11/1.E, R3.2, R6.2; no longer R14.2, R17.2, R2/1.E
- net LINE_IN_R: now also R10/1.E, R4.2, R5.2; no longer R1/1.E, R12.2, R52.2
- net N$1: now also C8.1, IC2G$4.IN-, R11/1.S, R11/2.A; no longer C1.1, IC4G$4.IN-, R1/1.S, R1/2.A
- net N$10: now also R4.1; no longer R12.1
- net N$11: now also R3.1; no longer R14.1
- net N$12: now also IC2G$1.IN-, R12.1, R13.2; no longer IC4G$1.IN-, R10.1, R9.2
- net N$13: now also IC3G$2.IN-, R23.2, R26.1; no longer IC1G$2.IN-, R18.2, R19.1
- net N$14: now also IC3G$1.IN-, R22.2, R25.1; no longer IC1G$1.IN-, R20.2, R21.1
- net N$15: now also IC3G$4.IN-, R27.2, R35.1; no longer IC1G$4.IN-, R22.2, R23.1
- net N$16: now also IC3G$4.OUT, R35.2, R37.1; no longer IC1G$4.OUT, R23.2, R24.1
- net N$17: now also IC3G$4.IN+, R28.2, R31.1; no longer IC1G$4.IN+, R25.2, R27.1
- net N$18: now also IC3G$3.IN-, R29.2, R36.1; no longer IC1G$3.IN-, R28.2, R29.1
- net N$19: now also IC3G$3.OUT, R36.2, R38.1; no longer IC1G$3.OUT, R29.2, R30.1
- net N$2: now also C7.1, IC2G$3.IN-, R10/1.S, R10/2.A; no longer C2.1, IC4G$3.IN-, R2/1.S, R2/2.A
- net N$20: now also IC3G$3.IN+, R30.2; no longer IC1G$3.IN+, R31.2
- net N$21: now also IC3G$1.OUT, R25.2, R29.1; no longer IC1G$1.OUT, R21.2, R25.1
- net N$22: now also IC3G$2.OUT, R26.2, R27.1, R30.1; no longer IC1G$2.OUT, R19.2, R22.1, R31.1
- net N$23: now also C20.1, IC3G$1.IN+, R24.2; no longer C8.1, IC1G$1.IN+, R34.2
- net N$24: now also C21.1, R23.1; no longer C9.1, R18.1
- net N$25: now also IC4G$2.IN-, R40.2, R43.1; no longer IC3G$2.IN-, R35.2, R36.1
- net N$26: now also IC4G$1.IN-, R39.2, R42.1; no longer IC3G$1.IN-, R37.2, R38.1
- net N$27: now also IC4G$4.IN-, R44.2, R52.1; no longer IC3G$4.IN-, R39.2, R40.1
- net N$28: now also IC4G$4.OUT, R52.2, R54.1; no longer IC3G$4.OUT, R40.2, R41.1
- net N$29: now also IC4G$4.IN+, R45.2, R48.1; no longer IC3G$4.IN+, R42.2, R44.1
- net N$3: now also C12.1, C8.2, IC2G$4.OUT, R14.2, R17.1; no longer C1.2, C7.1, IC4G$4.OUT, R55.2, R6.1
- net N$30: now also IC4G$3.IN-, R46.2, R53.1; no longer IC3G$3.IN-, R45.2, R46.1
- net N$31: now also IC4G$3.OUT, R53.2, R55.1; no longer IC3G$3.OUT, R46.2, R47.1
- net N$32: now also IC4G$3.IN+, R47.2; no longer IC3G$3.IN+, R48.2
- net N$33: now also IC4G$1.OUT, R42.2, R46.1; no longer IC3G$1.OUT, R38.2, R42.1
- net N$34: now also IC4G$2.OUT, R43.2, R44.1, R47.1; no longer IC3G$2.OUT, R36.2, R39.1, R48.1
- net N$35: now also C27.1, IC4G$1.IN+, R41.2; no longer C15.1, IC3G$1.IN+, R51.2
- net N$36: now also C28.1, R40.1; no longer C16.1, R35.1
- net N$37: now also C18.2; no longer C27.2
- net N$39: now also R2.1; no longer R15.1
- net N$4: now also C11.1, C7.2, IC2G$3.OUT, R15.2, R16.1; no longer C2.2, C4.1, IC4G$3.OUT, R11.2, R3.1
- net N$40: now also R1.1; no longer R13.1
- net N$41: now also C1.1, C2.1, C3.1, D1.2, IC1.IN; no longer C31.1, C32.1, C33.1, D5.2, IC2.IN
- net N$42: now also R11/2.S, R14.1; no longer R1/2.S, R55.1
- net N$43: now also IC1.FB, R8.1, R9.2; no longer IC2.FB, R53.2, R54.1
- net N$44: now also C19.2; no longer C26.2
- net N$5: now also C14.1, R16.2, R20.1; no longer C3.1, R3.2, R4.1
- net N$6: now also R10/2.S, R15.1; no longer R11.1, R2/2.S
- net N$7: now also C15.1, R17.2, R21.1; no longer C6.1, R6.2, R7.1
- net N$8: now also C11.2, C16.1, R18.2; no longer C4.2, C5.1, R5.2
- net N$9: now also C12.2, C17.1, R19.2; no longer C22.1, C7.2, R8.2
- net R: now also R5.1; no longer R52.1
- net SCHIRMUNG: now also R7.1; no longer R16.1
- net VREF_2V: now also IC2G$1.IN+, IC2G$1.OUT, IC4G$2.IN+, R22.1, R24.1, R34.2, R39.1, R41.1, R51.2; no longer IC1G$2.IN+, IC4G$1.IN+, IC4G$1.OUT, R20.1, R26.2, R34.1, R37.1, R43.2, R51.1
